Commit message: Release 0.3.3: joint names export, LIN retiming, and FK transform fix.
Adds RobotModel.JointNames, named trajectory JSON export, URDF FK cross-checks, and retimed Cartesian LIN durations; fixes column-major transform composition.

Co-authored-by: Cursor <cursoragent@cursor.com>

File: tests/fixtures/prismatic_lift.urdf (robot description, URDF)
Before this commit: robot prismatic_lift, 3 links, 2 joints
Links:
- link lift_link: geometry visual box size=0.12 0.12 0.25
- link tip_link: geometry visual box size=0.15 0.04 0.04

File: tests/fixtures/two_link.urdf (robot description, URDF)
Before this commit: robot two_link, 3 links, 2 joints
Links:
- link link1: geometry visual box size=0.2 0.04 0.04
- link tip_link: geometry visual sphere radius=0.035
