Commit message: Release 0.4.0: attach, planning groups, Motus.Native stubs, Rhino desktop path.
Adds PlanningContext/AttachedBody, SRDF groups with ForGroup planning tests,
unified motus_native (OMPL+FCL), native path simplification, group-aware RRT,
toolCollision presets, official ur10e.srdf, CI stub/full-native profiles,
URDF mesh path containment, and 83 passing tests.

Co-authored-by: Cursor <cursoragent@cursor.com>

File: tests/fixtures/ur5e_collision.urdf (robot description, URDF)
Before this commit: robot ur5e_minimal, 7 links, 6 joints
Links:
- link tool0: geometry collision box size=0.04 0.04 0.08
