Commit message: Add HolonomicSE3 hover foundation and quadrotor free-flyer fixture.
HoverHandoff bounds, base-frame attach, and station-hold support GH aerial preview; free_flyer URDF carries multi-visual silhouette for Preview.

Co-authored-by: Cursor <cursoragent@cursor.com>

File: tests/fixtures/aerial/free_flyer_box.urdf (robot description, URDF)
Before this commit: robot free_flyer_box, 1 links, 0 joints
Links:
- link body: mass 0.5 -> 0.8; geometry collision box size=0.22 0.22 0.08; visual box size=0.02 0.16 0.015
