Commit message: Bamboo viewer: full, physically-true Motus collision (pole, strut, ground, mount, self)
- bamboo_icd.urdf regenerated (tools/bamboo/gen_bamboo_urdf.py): arm hangs from a fixed
  pole_hang joint so URDF link frames == viewer Three.js groups; collision boxes == drawn boxes.
  Tests assert Motus FK == drawn chain to 1e-9 m.
- BambooIcdCell: Motus CollisionScene with pole + strut (tessellated meshes), ground slab,
  mount parts; strut rests at the pick object, is captured at its real jaw offset, stays where
  released; only the R-grip jaw plates may touch it while gripping.
- BambooMotionScan: samples the motion (<=0.5 deg/check), first Motus contact + last clear sample;
  /bamboo play/scrub park there and tint the parts Motus names. viewer.js draws from the cell
  description (no JS collision).
- Motus.Geometry: exact narrow phase (OBB SAT, triangle-OBB SAT, mesh vs primitives per triangle),
  RobotMeshCollisionChecker.FindContacts (named pairs), geometry-level allowed pairs, configurable
  self-collision gap, URDF <collision name>.
- Planner floor heuristics demoted to IK-branch preference; BambooIcdIk adapts planar IK for
  TaskPathValidator.
- Tests: default path passes; grasp -1.5 mm (neck<->strut), release -10 mm (strut<->ground),
  swing through pole, fold into mount, dive to ground, self-collision all fail with named contacts.

File: src/Motus.Viewer/wwwroot/fixtures/bamboo_icd/bamboo_icd.urdf (robot description, URDF)
Before this commit: robot bamboo_icd, 8 links, 7 joints
Links:
- removed link gripper_link
- added link mount; collision box size=0.0045 0.03 0.024; collision box size=0.0045 0.03 0.024
- link base_link: geometry 
- link link_1: geometry collision box size=0.012 0.064 0.016; collision box size=0.046 0.029 0.034
- link link_2: geometry collision box size=0.012 0.072 0.016; collision box size=0.041 0.061 0.04
- link link_3: geometry collision box size=0.012 0.072 0.016; collision box size=0.041 0.061 0.04
- link link_4: geometry collision box size=0.012 0.072 0.016; collision box size=0.041 0.061 0.04
- link link_5: geometry collision box size=0.0045 0.02 0.022; collision box size=0.0045 0.02 0.022
Joints:
- removed joint gripper_joint
- added joint pole_hang: type fixed, parent base_link, child mount, origin xyz=0 0 0.4 rpy=1.5707963267948966 0 1.5707963267948966
- joint joint_1: axis 0 0 1 -> 0 1 0; limit lower=-2.967 upper=2.967 effort=100 velocity=2.0 -> lower=-2.967060 upper=2.967060 effort=10 velocity=2.0; origin xyz=0 0 0.1 rpy=0 0 0 -> xyz=0 -0.03 0 rpy=0 0 0; parent base_link -> mount
- joint joint_2: limit lower=-1.571 upper=1.571 effort=100 velocity=2.0 -> lower=-1.570796 upper=1.570796 effort=10 velocity=2.0; origin xyz=0 0 0.3 rpy=0 0 0 -> xyz=0 -0.08 0 rpy=0 0 0
- joint joint_3: limit lower=-2.356 upper=2.356 effort=100 velocity=2.0 -> lower=-2.356194 upper=2.356194 effort=10 velocity=2.0; origin xyz=0 0 0.25 rpy=0 0 0 -> xyz=0 -0.088 0 rpy=0 0 0
- joint joint_4: limit lower=-1.571 upper=1.571 effort=100 velocity=2.0 -> lower=-1.570796 upper=1.570796 effort=10 velocity=2.0; origin xyz=0 0 0.25 rpy=0 0 0 -> xyz=0 -0.088 0 rpy=0 0 0
- joint joint_5: axis 0 0 1 -> 0 1 0; limit lower=-2.967 upper=2.967 effort=50 velocity=2.0 -> lower=-2.967060 upper=2.967060 effort=10 velocity=2.0; origin xyz=0 0 0.2 rpy=0 0 0 -> xyz=0 -0.088 0 rpy=0 0 0
- joint tool_joint: origin xyz=0 0 0.02 rpy=0 0 0 -> xyz=0 -0.046 0 rpy=0 0 0; parent gripper_link -> link_5
