Commit message: WIP bamboo-truss: L-grip opened on one side (+y) for side clamping (deviation from ICD URDF); goal-driven brachiation search; RRT retries; open-side slot test

File: tests/fixtures/bamboo_icd/bamboo_icd.urdf (robot description, URDF)
Before this commit: robot bamboo_icd, 8 links, 7 joints
Links:
- link mount: geometry collision box size=0.0045 0.03 0.024; collision box size=0.0045 0.03 0.024
